File: pcb/picobox/picobox.kicad_sch (KiCad schematic)
At the start: 11 parts, among them J1 OLED, SW1 SW_SPDT, U1 Pico

Commit message: finish schematic
Parts:
- added C1: 100n, Capacitor_THT:C_Disc_D5.0mm_W2.5mm_P5.00mm, symbol Device:C
- A1: renamed from A; footprint (none) -> Button_Switch_THT:SW_PUSH_6mm
- B1: renamed from B; footprint (none) -> Button_Switch_THT:SW_PUSH_6mm
- BT1: footprint (none) -> Battery:BatteryHolder_Keystone_2462_2xAA
- DOWN1: renamed from DOWN; footprint (none) -> Button_Switch_THT:SW_PUSH_6mm
- HOME1: renamed from HOME; footprint (none) -> Button_Switch_THT:SW_PUSH_6mm
- J1: footprint (none) -> Connector_PinHeader_2.54mm:PinHeader_1x04_P2.54mm_Horizontal
- LEFT1: renamed from LEFT; footprint (none) -> Button_Switch_THT:SW_PUSH_6mm
- RIGHT1: renamed from RIGHT; footprint (none) -> Button_Switch_THT:SW_PUSH_6mm
- SW1: footprint (none) -> Button_Switch_THT:SW_Slide_SPDT_Straight_CK_OS102011MS2Q
- UP1: renamed from UP; footprint (none) -> Button_Switch_THT:SW_PUSH_6mm
Connections:
- net GND: now reaches A1.2, B1.2, DOWN1.2, HOME1.2, J1.1 (Pin_1), LEFT1.2, RIGHT1.2, UP1.2
- net GND: now also BT1.2 (-), C1.2; no longer U1.38 (GND)
- net at J1.2 (Pin_2), U1.36 (3V3): now also C1.1
- net at U1.3 (GND): no longer BT1.2 (-)
- no-connect marks 0 -> 33
