File: pcb/picobox/picobox.kicad_pcb (KiCad board)
At the start: 2 copper layers, 87.4 x 116.8 mm, 12 parts, among them J1 OLED, SW1 SW_SPDT, U1 Pico

Commit message: finish pcb design
Parts:
- moved HOME1 9.69 mm to (198.9, 140.2)
Routing:
- net Net-(J1-Pin_2): track 0.00 -> 153.8 mm
- net Net-(U1-GPIO9): track 0.00 -> 129.6 mm, vias 0 -> 2
- net Net-(U1-GPIO12): track 0.00 -> 126.4 mm, vias 0 -> 2
- net Net-(U1-GPIO7): track 0.00 -> 125.0 mm, vias 0 -> 8
- net Net-(J1-Pin_3): track 0.00 -> 114.9 mm, vias 0 -> 2
- net Net-(J1-Pin_4): track 0.00 -> 111.7 mm, vias 0 -> 4
- net Net-(U1-GPIO8): track 0.00 -> 100.2 mm, vias 0 -> 6
- net Net-(U1-GPIO11): track 0.00 -> 99.6 mm, vias 0 -> 4
- net Net-(U1-GPIO6): track 0.00 -> 95.9 mm, vias 0 -> 2
- net Net-(U1-GPIO10): track 0.00 -> 88.6 mm, vias 0 -> 2
- net Net-(SW1-B): track 0.00 -> 61.1 mm
- net Net-(BT1-+): track 0.00 -> 24.5 mm, vias 0 -> 2
- added copper zone on B.Cu, net GND
Other:
- board text added: "PicoBox Mark I"
