File: pcb/picobox/picobox.kicad_pcb (KiCad board)
At the start: 2 copper layers, 87.4 x 116.8 mm, 12 parts, among them J1 OLED, SW1 SW_SPDT, U1 Pico

Commit message: move pico to the left so usb is accessible
Parts:
- moved U1 17.0 mm to (149.6, 48.4)
Routing:
- net Net-(SW1-B): track 61.1 -> 167.3 mm, vias 0 -> 2
- net Net-(U1-GPIO7): track 125.0 -> 100.8 mm, vias 8 -> 4
- net Net-(U1-GPIO11): track 99.6 -> 119.5 mm, vias 4 -> 6
- net Net-(U1-GPIO12): track 126.4 -> 146.2 mm, vias 2 -> 8
- net Net-(U1-GPIO8): track 100.2 -> 82.9 mm, vias 6 -> 2
- net Net-(U1-GPIO6): track 95.9 -> 80.0 mm
- net Net-(U1-GPIO10): track 88.6 -> 104.2 mm, vias 2 -> 4
- net Net-(U1-GPIO9): track 129.6 -> 115.4 mm
- net Net-(J1-Pin_4): track 111.7 -> 98.1 mm, vias 4 -> 6
- net Net-(J1-Pin_3): track 114.9 -> 101.6 mm, vias 2 -> 4
- net Net-(J1-Pin_2): track 153.8 -> 162.6 mm, vias 0 -> 4
- net unconnected-(U1-GPIO14-Pad19)_1: track 0.00 -> 1.56 mm
